File: WiringDiagram/KiCad/BuggyElectrical.kicad_sch (KiCad schematic)
At the start: 12 parts

Commit message: Laptop Update
Parts:
- removed 3.BrakeLight, AV-Video_BackUpCam, LicensePlateLight, Power_BackUpCam: JST_01x02_Male, symbol Connector:Conn_01x02_Male
- removed AV-Video_BackUpCam: JST_01x03_Female, symbol Connector:Conn_01x03_Female
- removed OffroadRearLeft, OffroadRearRight, Reverse+RearLeft, Reverse+RearRight: SuperSeal_01x02_Male, symbol Connector:Conn_01x02_Male
- removed RearLeftLight, RearRightLight: SuperSeal_01x06_Male, symbol Connector:Conn_01x06_Male
- removed Rear_Wiring_Connector: DT_02x06_Female, symbol Connector_Generic:Conn_02x06_Counter_Clockwise
Other:
- added sheet AHKHarness (AHKHarness.kicad_sch)
- added sheet RearWiringHarnessTop (RearWiringHarness.kicad_sch)
- added sheet RelaySafetyBox (RelaySafetyBox.kicad_sch)
- note removed: "1. Free 2. Rückfahrlicht/Kamera 3. Rücklicht Links/Kennzeichen (überprüfen) 4. Blinker Links (überprüfen) 5. Nebelschlussleuchte 6. Bremslicht Links 7. Off-road Hinten 8. Zusatz Rückfahrlicht 9. Bremslicht Rechts 10. Rücklicht Rechts 11. Blinker Rechts 12. Free"
- note removed: "Male/Female is about the Crimped inner part, not the Plug itself"
- note removed: "Rear Wiring Harness"
